Commit message: Second commit

File: resources/robots/tita_airbot/urdf/robot.urdf (robot description, URDF)
Before this commit: robot tita, 22 links, 21 joints
Links:
- added link G2_link1, mass 0.078003; collision mesh filename=../meshes/arm/G2/collision/link1.STL; visual mesh filename=../meshes/arm/G2/visual/link1.STL
- added link G2_link2, mass 0.078003; collision mesh filename=../meshes/arm/G2/collision/link2.STL; visual mesh filename=../meshes/arm/G2/visual/link2.STL
- added link end_link, mass 0.605
- added link flange, mass 0.0206; collision mesh filename=../meshes/arm/flange/collision/flange.obj scale=1. 1. 1.; visual mesh filename=../meshes/arm/flange/visual/flange.obj scale=1. 1. 1.
- added link link_G2_base, mass 0.26507; collision mesh filename=../meshes/arm/G2/collision/base_link.STL; visual mesh filename=../meshes/arm/G2/visual/base_link.STL
- added link rotate_motor
- link arm_base_link: mass 0.775915004746176 -> 0.683; geometry collision mesh filename=../meshes/arm/airbot_play_v3_1/collision/base_link.STL; visual mesh filename=../meshes/arm/airbot_play_v3_1/visual/base_link.STL
- link link1: mass 0.557107161361679 -> 0.609; geometry visual mesh filename=../meshes/arm/airbot_play_v3_1/visual/link1.STL
- link link2: mass 0.646248710360021 -> 0.902; geometry visual mesh filename=../meshes/arm/airbot_play_v3_1/visual/link2.STL
- link link3: mass 0.445563107671385 -> 0.683; geometry visual mesh filename=../meshes/arm/airbot_play_v3_1/visual/link3.STL
- link link4: mass 0.345884858675684 -> 0.358; geometry visual mesh filename=../meshes/arm/airbot_play_v3_1/visual/link4.STL
- link link5: mass 0.18663635710924 -> 0.403; geometry visual mesh filename=../meshes/arm/airbot_play_v3_1/visual/link5.STL
- link link6: mass 0.17462115508378 -> 0.118; geometry visual mesh filename=../meshes/arm/airbot_play_v3_1/visual/link6.STL
Joints:
- removed joint arm_base
- removed joint arm_joint1
- removed joint arm_joint2
- removed joint arm_joint3
- removed joint arm_joint4
- removed joint arm_joint5
- removed joint arm_joint6
- added joint G2_joint1: type fixed, parent link_G2_base, child G2_link1, origin xyz=0.0736 0.05 -0.015 rpy=0 1.5708 0, axis 0 1 0, limit lower=-0.034 upper=0 effort=3 velocity=1, mimic joint=gripper_joint multiplier=-0.034 offset=0
- added joint G2_joint2: type fixed, parent link_G2_base, child G2_link2, origin xyz=0.0736 -0.05 -0.015 rpy=0 1.5708 0, axis 0 1 0, limit lower=0 upper=0.034 effort=3 velocity=1, mimic joint=gripper_joint multiplier=0.034 offset=0
- added joint arm_to_flange: type fixed, parent link6, child flange, origin xyz=0 0 0 rpy=0 0 0
- added joint end_joint: type fixed, parent flange, child end_link, origin xyz=0.1602 0 0 rpy=0 0 0
- added joint gripper_connector: type fixed, parent flange, child link_G2_base, origin xyz=0.009 0 0 rpy=0 0 0
- added joint gripper_joint: type fixed, parent link_G2_base, child rotate_motor, origin xyz=0 0 0 rpy=0 0 0, axis 0 0 1, limit lower=0 upper=1 effort=20 velocity=3.1415926
- added joint joint_arm_1: type revolute, parent arm_base_link, child link1, origin xyz=0 0 0.1117 rpy=0 0 0, axis 0 0 1, limit lower=-3.151 upper=2.089 effort=20 velocity=2.
- added joint joint_arm_2: type revolute, parent link1, child link2, origin xyz=0 0 0 rpy=-1.5691 -0.38673 3.1409, axis 0 0 1, limit lower=-2.963 upper=0.181 effort=20 velocity=2.
- added joint joint_arm_3: type revolute, parent link2, child link3, origin xyz=0.27009 0 0 rpy=0 0.0015895 1.9575, axis 0 0 1, limit lower=-0.094 upper=3.161 effort=20 velocity=6.8
- added joint joint_arm_4: type revolute, parent link3, child link4, origin xyz=8.2128E-05 0.29015 0 rpy=-1.5708 -1.5708 0, axis 0 0 1, limit lower=-3.012 upper=3.012 effort=3 velocity=6.8
- added joint joint_arm_5: type revolute, parent link4, child link5, origin xyz=0 0 0 rpy=1.5708 0 0, axis 0 0 1, limit lower=-1.859 upper=1.859 effort=3 velocity=6.8
- added joint joint_arm_6: type revolute, parent link5, child link6, origin xyz=0 0.0864 0 rpy=0 0 1.5708, axis 1 0 0, limit lower=-3.017 upper=3.017 effort=3 velocity=6.8
- added joint joint_to_arm_base: type fixed, parent base_link, child arm_base_link, origin xyz=0.01447 0 0.1573 rpy=0 0 0, axis 0 0 1
